File: Soil Power Sensor.brd (EAGLE design)
At the start: 94 x 67 mm, 92 parts, among them IC1 TPD2E2U06DCK, J1 12401832E402A, U1 MAX9943ATT+, U10 FT234XD, U11 ESP32-C3-MINI-1-N4, U2 INA296A5, U3 THS4532, U4 FSA2466, U5 MAX11201A, U6 REF2033, U7 TLV1117LV33, U8 LM27761DSG, U9 WIO E5, X1 Voltage, X2 Current, X3 GND, X4 SDI, X5 SMA-142-0701-801/806

Commit message: Closes #2
Parts:
- removed C12, C17: 4.7uF, rcl:C0603
- removed C13, C14: NC, rcl:C0603
- removed C15, C16, C18: 0.1uF, rcl:C0603
- removed C7, C9: 1uF, rcl:C0603
- removed E1: MI0805K601R-10, Soil Power Sensor:FB_MI0805K601R-10
- removed IC1: TPD2E2U06DCK, Soil Power Sensor:SOT65P210X110-3N
- removed J1: 12401832E402A, Connector_USB:12401832E402A
- removed R12, R15: 5.1k, rcl:R0603
- removed R16, R17, R18, R20, R21, R22, R23: 0, rcl:R0603
- removed S1: STM32 Reset, switch-omron:B3F-10XX
- removed U10: FT234XD, Soil Power Sensor:SON45P300X300X80-13N
- removed U9: WIO E5, Soil Power Sensor:MODULE28P-1.25-12X12X2.5MM
- removed X5: SMA-142-0701-801/806, con-coax:J502-ND-142-0701-801/806
- U7: value TLV1117LV33 -> WIO-E5_MINI; device Soil Power Sensor:SOT230P700X180-4N -> Soil Power Sensor:WIO-E5_MINI
- moved U7 85.2 mm to (-53.8, 37.3)
Connections:
- removed net N$10: R20.1, U10.8
- removed net N$11: R21.1, U10.11
- removed net N$12: R22.1, U10.10
- removed net N$13: R23.1, U10.7
- removed net N$14: C18.1, U10.2, U10.3, U10.9
- removed net N$15: C16.1, C17.1, E1.2, U10.4
- removed net N$22: U9.23, X4.1
- removed net N$6: J1.A5, R12.2
- removed net N$7: J1.B5, R15.1
- removed net PB6/TX: R23.2, U9.10
- removed net PB7/RX: R22.2, U9.9
- removed net STMR_D_N: R18.2, U10.1
- removed net STMR_D_P: R17.2, U10.12
- removed net STM_D_N: IC1.2, J1.A7, J1.B7, R18.1
- removed net STM_D_P: IC1.1, J1.A6, J1.B6, R17.1
- net +3V3: now also U7.P22; no longer C12.1, C9.1, U7.2, U7.4, U9.1
- net ESP32_EN: no longer U9.21
- net ESP32_RXD0: no longer U9.18
- net ESP32_TXD0: no longer U9.19
- net GND: now also U7.P0, U7.P18; no longer C12.2, C13.2, C14.2, C15.2, C16.2, C17.2, C18.2, C7.1, C9.2, IC1.3, J1.A1, J1.A12, J1.B1, J1.B12, J1.SH1, J1.SH2, J1.SH3, J1.SH4, R12.1, R15.2, S1.1, S1.2, U10.13, U10.5, U7.1, U9.14, U9.16, U9.2, U9.22, X5.G@1, X5.G@2, X5.G@3, X5.G@4
- net JTCK: no longer U9.4
- net JTDI: no longer U9.6
- net JTMS: no longer U9.3
- net N$2: now also U7.P11, X4.1; no longer C14.1, R16.2, X5.1
- net N$3: now also R13.1, R14.2; no longer C13.1, R16.1, U9.15
- net N$34: now also U7.P14; no longer R13.1, R14.2, U9.27
- net PB13/SPI2_SCK: no longer U9.24
- net PB14/SPI2_MISO: no longer U9.26
- net PB3/RTS/JTDO: no longer R20.2, U9.8
- net PB4/CTS/JNTRST: no longer R21.2, U9.7
- net PB9/SPI2_NSS: no longer U9.25
- net PC0: no longer U9.13
- net PC1: no longer U9.12
- net RST: no longer C15.1, S1.3, S1.4, U9.17
- net VCC: no longer C7.2, U7.3
- net VUSB: now also U7.P23; no longer E1.1, J1.A4, J1.A9, J1.B4, J1.B9
Routing:
- net N$22: track 86.2 -> 0.00 mm, vias 2 -> 0
- net PB6/TX: track 46.3 -> 0.00 mm, vias 2 -> 0
- net RST: track 43.7 -> 9.81 mm
- net PB7/RX: track 33.8 -> 0.00 mm, vias 2 -> 0
- net STM_D_P: track 32.3 -> 0.00 mm, vias 2 -> 0
- net STM_D_N: track 27.1 -> 0.00 mm, vias 2 -> 0
- net N$14: track 24.0 -> 0.00 mm, vias 2 -> 0
- net VUSB: track 119.3 -> 100.6 mm
- net N$15: track 16.5 -> 0.00 mm
- net +3V3: track 231.2 -> 217.1 mm
- net STMR_D_P: track 12.0 -> 0.00 mm
- net N$7: track 10.6 -> 0.00 mm, vias 2 -> 0
- net N$2: track 10.6 -> 0.00 mm
- net N$3: track 15.8 -> 5.76 mm
- net N$34: track 8.22 -> 0.00 mm
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
Commit message: Closes #3
Parts:
- removed C21, C22: NC, rcl:C0603
- removed JP4: STM32 JTAG, pinhead:2X10
- removed JP5: ESP32 JTAG, pinhead:2X10
- removed JP6: USB, jumper:JP1
- removed R19, R27, R28: 0, rcl:R0603
- added D1, D2: ARM10_DEBUG, Soil Power Sensor:ARM10_DEBUG
Connections:
- removed net D_N: R27.1, U11.26
- removed net D_P: R28.1, U11.27
- removed net IO4/TMS: JP5.7, U11.18
- removed net IO5/TDI: JP5.5, U11.19
- removed net IO6/TCK: JP5.9, U11.20
- removed net IO7/TDO: JP5.13, U11.21
- removed net JTCK: JP4.9
- removed net JTDI: JP4.5
- removed net JTMS: JP4.7
- removed net N$39: C21.1, JP6.1, R27.2
- removed net N$40: C22.1, JP6.2, R28.2
- removed net NRST: JP4.15, R19.2
- removed net PB3/RTS/JTDO: JP4.13
- removed net PB4/CTS/JNTRST: JP4.3
- removed net RST: R19.1
- new net ESP32_TCK: D2.TCK/SWDCLK, U11.20
- new net ESP32_TDI: D2.TDI, U11.19
- new net ESP32_TDO: D2.TDO/SWO, U11.21
- new net ESP32_TMS: D2.TMS/SWDIO, U11.18
- new net STM_SWDCLK: D1.TCK/SWDCLK, U7.P20
- new net STM_SWDIO: D1.TMS/SWDIO, U7.P21
- new net STM_SWO: D1.TDO/SWO, U7.P4
- net +3V3: now also D1.VCC, D2.VCC; no longer JP4.1, JP4.2, JP5.1, JP5.2
- net ESP32_NRST: no longer JP5.15
- net GND: now also D1.GND@3, D1.GND@5, D1.GND@9, D2.GND@3, D2.GND@5, D2.GND@9; no longer C21.2, C22.2, JP4.10, JP4.12, JP4.14, JP4.16, JP4.18, JP4.20, JP4.4, JP4.6, JP4.8, JP5.10, JP5.12, JP5.14, JP5.16, JP5.18, JP5.20, JP5.4, JP5.6, JP5.8
Routing:
- net PB3/RTS/JTDO: track 77.2 -> 0.00 mm, vias 3 -> 0
- net IO7/TDO: track 57.7 -> 0.00 mm, vias 1 -> 0
- net ESP32_TDO: track 0.00 -> 55.9 mm, vias 0 -> 1
- net IO6/TCK: track 52.3 -> 0.00 mm, vias 1 -> 0
- net ESP32_TCK: track 0.00 -> 50.9 mm, vias 0 -> 1
- net NRST: track 49.6 -> 0.00 mm
- net IO4/TMS: track 48.5 -> 0.00 mm, vias 1 -> 0
- net PB4/CTS/JNTRST: track 46.7 -> 0.00 mm, vias 2 -> 0
- net IO5/TDI: track 46.0 -> 0.00 mm, vias 1 -> 0
- net ESP32_TMS: track 0.00 -> 44.2 mm, vias 0 -> 1
- net ESP32_TDI: track 0.00 -> 42.2 mm, vias 0 -> 1
- net JTCK: track 36.5 -> 0.00 mm, vias 1 -> 0
- net JTMS: track 34.1 -> 0.00 mm, vias 1 -> 0
- net JTDI: track 28.2 -> 0.00 mm, vias 1 -> 0
- net +3V3: track 217.1 -> 193.6 mm
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
Commit message: Closes #7
Parts:
- removed IN, IP, VBUF, VCM, VN, VP: TPB1,27, testpad:B1,27
- added -3V3, 3V3, REF_1V65, REF_3V3, VBAT, VCC, VUSB: TPB1,27, testpad:B1,27
Connections:
- net +3V3: now also 3V3.TP
- net -3V3: now also -3V3.TP
- net CURRENT_N: no longer IN.TP
- net CURRENT_P: no longer IP.TP
- net N$19: now also VBAT.TP
- net N$46: no longer VCM.TP
- net N$8: no longer VBUF.TP
- net REF+1V65: now also REF_1V65.TP
- net REF+3V3: now also REF_3V3.TP
- net VCC: now also VCC.TP
- net VOLTAGE_N: no longer VN.TP
- net VOLTAGE_P: no longer VP.TP
- net VUSB: now also VUSB.TP
Routing:
- net N$8: track 30.4 -> 27.6 mm
- net N$46: track 71.2 -> 68.7 mm
- net VOLTAGE_N: track 41.0 -> 38.5 mm
- net VOLTAGE_P: track 46.2 -> 44.3 mm
- net CURRENT_P: track 47.2 -> 46.1 mm
- net CURRENT_N: track 38.9 -> 38.3 mm

Commit message: Closes #14
Parts:
- removed U1: MAX9943ATT+, Soil Power Sensor:TDFN300X300X75-6N
- added U9: MAX9944ASA, Soil Power Sensor:SOIC127P600X155-8N
Connections:
- new net N$4: R3.1, U9.6, U9.7
- net +3V3: now also U9.8; no longer U1.6
- net -3V3: now also U9.4; no longer U1.2
- net N$1: now also U9.3; no longer U1.3
- net N$46: now also U9.5; no longer R3.1
- net N$8: now also U9.1, U9.2; no longer U1.1, U1.4
Routing:
- net N$8: track 27.6 -> 18.6 mm
- net N$1: track 50.2 -> 41.2 mm
- net -3V3: track 17.6 -> 13.7 mm
- net N$46: track 68.7 -> 67.0 mm
- net +3V3: track 193.6 -> 193.1 mm
Changed lines of the file:
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@@
 <attribute name="REF" value="https://www.ti.com/product/REF2033" x="137.16" y="-63.5" size="1.778" layer="27" display="off"/>
-</element>
-<element name="U1" library="Soil Power Sensor" package="TDFN300X300X75-6N" value="MAX9943ATT+" x="30.48" y="48.26" smashed="yes">
-<attribute name="AUTHOR" value="John Madden &lt;jmadden173@pm.me&gt;" x="137.16" y="-38.1" size="1.778" layer="27" display="off"/>
-<attribute name="DATE_CREATED" value="2023-04-26" x="137.16" y="-38.1" size="1.778" layer="27" display="off"/>
-<attribute name="DATE_MODIFIED" value="2023-04-26" x="137.16" y="-38.1" size="1.778" layer="27" display="off"/>
-<attribute name="MFC" value="Analog Devices" x="137.16" y="-38.1" size="1.778" layer="27" display="off"/>
-<attribute name="MPN" value="MAX9943ATT+T" x="137.16" y="-38.1" size="1.778" layer="27" display="off"/>
-<attribute name="NAME" x="29.234" y="50.062" size="1.27" layer="25"/>
-<attribute name="REF" value="https://www.analog.com/en/products/MAX9943.html" x="137.16" y="-38.1" size="1.778" layer="27" display="off"/>
 </element>
 <element name="U11" library="Soil Power Sensor" package="XCVR_ESP32-C3-MINI-1-N4" value="ESP32-C3-MINI-1-N4" x="90.17" y="8.89" smashed="yes" rot="R270">
@@
 <attribute name="VALUE" x="-53.975" y="-71.882" size="0.0254" layer="27"/>
 </element>
+<element name="U9" library="Soil Power Sensor" package="SOIC127P600X155-8N" value="MAX9944ASA" x="-60.96" y="-66.04" smashed="yes">
+<attribute name="AUTHOR" value="John Madden &lt;jmadden173@pm.me&gt;" x="-60.96" y="-66.04" size="1.778" layer="27" display="off"/>
+<attribute name="DATE_CREATED" value="2023-04-05" x="-60.96" y="-66.04" size="1.778" layer="27" display="off"/>
+<attribute name="DATE_MODIFIED" value="2023-04-05" x="-60.96" y="-66.04" size="1.778" layer="27" display="off"/>
+<attribute name="MFC" value="Analog Devices" x="-60.96" y="-66.04" size="1.778" layer="27" display="off"/>
+<attribute name="MPN" value="MAX9944ASA+T" x="-60.96" y="-66.04" size="1.778" layer="27" display="off"/>
+<attribute name="NAME" x="-64.695" y="-62.865" size="1.27" layer="25"/>
+<attribute name="QTY" value="1" x="-60.96" y="-66.04" size="1.778" layer="27" display="off"/>
+<attribute name="REF" value="https://www.analog.com/en/products/max9944.html#product-overview" x="-60.96" y="-66.04" size="1.778" layer="27" display="off"/>
+<attribute name="VALUE" x="-64.695" y="-70.485" size="1.27" layer="27"/>
+</element>
 </elements>
 <signals>
@@
 <contactref element="U5" pad="6"/>
 <contactref element="U5" pad="7"/>
-<contactref element="U1" pad="6"/>
 <contactref element="U11" pad="3"/>
 <contactref element="R29" pad="2"/>
@@
 <wire x1="39.9768" y1="42.3192" x2="40.132" y2="42.164" width="0.1524" layer="1"/>
 <via x="40.132" y="42.164" extent="1-16" drill="0.35"/>
-<wire x1="31.98" y1="49.21" x2="31.98" y2="49.76" width="0.1524" layer="1"/>
 <wire x1="31.98" y1="49.76" x2="32.258" y2="50.038" width="0.1524" layer="1"/>
 <via x="32.258" y="50.038" extent="1-16" drill="0.35"/>
@@
 <contactref element="D2" pad="VCC"/>
 <contactref element="3V3" pad="TP"/>
-<wire x1="-50.8" y1="-27.94" x2="-53.34" y2="-71.12" width="0" layer="19" extent="1-1"/>
+<contactref element="U9" pad="8"/>
+<wire x1="-58.495" y1="-64.135" x2="-53.34" y2="-71.12" width="0" layer="19" extent="1-1"/>
+<wire x1="-50.8" y1="-27.94" x2="-58.495" y2="-64.135" width="0" layer="19" extent="1-1"/>
 <wire x1="-50.8" y1="-15.24" x2="-50.8" y2="-27.94" width="0" layer="19" extent="1-1"/>
 <wire x1="-30.848" y1="34.798" x2="-50.8" y2="-15.24" width="0" layer="19" extent="1-1"/>
@@
 <contactref element="X1" pad="1"/>
 <contactref element="JP2" pad="2"/>
-<contactref element="U1" pad="3"/>
 <wire x1="7.71090625" y1="40.82605" x2="4.98909375" y2="40.82605" width="0.1524" layer="1"/>
 <wire x1="6.35" y1="59.67485625" x2="6.35" y2="62.19" width="0.1524" layer="1"/>
@@
 <wire x1="17.72091875" y1="41.91" x2="16.51" y2="41.91" width="0.1524" layer="1"/>
 <wire x1="18.66071875" y1="40.9702" x2="17.72091875" y2="41.91" width="0.1524" layer="1"/>
-<wire x1="28.98" y1="47.31" x2="22.6402" y2="40.9702" width="0.1524" layer="1"/>
 <wire x1="22.6402" y1="40.9702" x2="18.66071875" y2="40.9702" width="0.1524" layer="1"/>
+<contactref element="U9" pad="3"/>
+<wire x1="16.51" y1="41.91" x2="-63.425" y2="-66.675" width="0" layer="19" extent="1-1"/>
 </signal>
 <signal name="N$46">
 <contactref element="JP2" pad="4"/>
 <contactref element="X1" pad="2"/>
-<contactref element="R3" pad="1"/>
 <wire x1="16.607675" y1="58.1406" x2="18.952325" y2="58.1406" width="0.1524" layer="1"/>
 <wire x1="18.952325" y1="58.1406" x2="19.5326" y2="57.560325" width="0.1524" layer="1"/>
@@
 <wire x1="37.338" y1="57.15" x2="37.338" y2="62.992" width="0.1524" layer="15"/>
 <via x="37.338" y="62.992" extent="1-16" drill="0.35"/>
-<wire x1="37.338" y1="62.992" x2="39.028" y2="62.992" width="0.1524" layer="1"/>
 <wire x1="13.97" y1="47.498" x2="17.78" y2="51.308" width="0.1524" layer="15"/>
+<contactref element="U9" pad="5"/>
+<wire x1="13.97" y1="45.72" x2="-58.495" y2="-67.945" width="0" layer="19" extent="1-1"/>
 </signal>
 <signal name="N$48">
@@
 </signal>
 <signal name="N$8">
-<contactref element="U1" pad="4"/>
-<contactref element="U1" pad="1"/>
 <contactref element="R2" pad="1"/>
-<wire x1="28.98" y1="49.21" x2="29.1117125" y2="49.21" width="0.1524" layer="1"/>
-<wire x1="31.98" y1="47.3517125" x2="31.98" y2="47.31" width="0.1524" layer="1"/>
 <via x="42.164" y="59.436" extent="1-16" drill="0.35"/>
 <wire x1="42.164" y1="59.436" x2="33.274" y2="50.546" width="0.1524" layer="15"/>
@@
 <via x="33.274" y="47.498" extent="1-16" drill="0.35"/>
 <wire x1="33.274" y1="47.498" x2="33.086" y2="47.31" width="0.1524" layer="1"/>
-<wire x1="33.086" y1="47.31" x2="31.98" y2="47.31" width="0.1524" layer="1"/>
 <wire x1="33.274" y1="47.498" x2="34.036" y2="48.26" width="0.1524" layer="1"/>
-<wire x1="32.50935" y1="50.6448" x2="32.8648" y2="50.28935" width="0.1524" layer="1"/>
-<wire x1="30.5465125" y1="50.6448" x2="32.50935" y2="50.6448" width="0.1524" layer="1"/>
-<wire x1="32.8648" y1="50.28935" x2="32.8648" y2="48.2365125" width="0.1524" layer="1"/>
-<wire x1="32.8648" y1="48.2365125" x2="31.98" y2="47.3517125" width="0.1524" layer="1"/>
-<wire x1="29.1117125" y1="49.21" x2="30.5465125" y2="50.6448" width="0.1524" layer="1"/>
 <wire x1="42.164" y1="59.436" x2="42.33" y2="59.602" width="0.1524" layer="1"/>
 <wire x1="42.33" y1="59.602" x2="42.33" y2="60.96" width="0.1524" layer="1"/>
+<contactref element="U9" pad="1"/>
+<contactref element="U9" pad="2"/>
+<wire x1="-63.425" y1="-65.405" x2="-63.425" y2="-64.135" width="0" layer="19" extent="1-1"/>
+<wire x1="33.086" y1="47.31" x2="-63.425" y2="-64.135" width="0" layer="19" extent="1-1"/>
 </signal>
 <signal name="-3V3">
-<contactref element="U1" pad="2"/>
 <contactref element="U8" pad="4"/>
 <contactref element="C11" pad="1"/>
@@
 <wire x1="28.84" y1="53.34" x2="26.3" y2="55.88" width="0.1524" layer="1"/>
 <wire x1="26.3" y1="55.88" x2="26.25" y2="55.88" width="0.1524" layer="1"/>
-<wire x1="28.98" y1="48.26" x2="26.25" y2="50.99" width="0.1524" layer="1"/>
 <wire x1="26.25" y1="50.99" x2="26.25" y2="55.88" width="0.1524" layer="1"/>
 <contactref element="-3V3" pad="TP"/>
-<wire x1="28.98" y1="48.26" x2="-53.34" y2="-55.88" width="0" layer="19" extent="1-1"/>
+<contactref element="U9" pad="4"/>
+<wire x1="-53.34" y1="-55.88" x2="-63.425" y2="-67.945" width="0" layer="19" extent="1-1"/>
+<wire x1="26.25" y1="50.99" x2="-53.34" y2="-55.88" width="0" layer="19" extent="1-1"/>
 </signal>
 <signal name="VCC">
@@
 <wire x1="-30.848" y1="29.718" x2="-46.77" y2="-16.51" width="0" layer="19" extent="1-1"/>
 </signal>
+<signal name="N$4">
+<contactref element="U9" pad="6"/>
+<contactref element="U9" pad="7"/>
+<contactref element="R3" pad="1"/>
+<wire x1="-58.495" y1="-65.405" x2="-58.495" y2="-66.675" width="0" layer="19" extent="1-1"/>
+<wire x1="39.028" y1="62.992" x2="-58.495" y2="-65.405" width="0" layer="19" extent="1-1"/>
+</signal>
 </signals>
