File: Soil Power Sensor.sch (EAGLE design)
At the start: 64 parts, among them U1 ADS1219IRTER, U11 ESP32-C3-MINI-1-N4, U2 INA296A5, U3 THS4532, U6 REF2033, U7 WIO-E5_MINI, U8 LM27761DSG, U9 MAX9944ASA, X1 Voltage, X2 Current, X3 GND, X4 SDI

Commit message: Closes #4
Parts:
- removed C11: 2.2uF, rcl:C-EUC0603
- removed R10: 169k, rcl:R-US_R0603
- removed R11: 100k, rcl:R-US_R0603
- removed U8: LM27761DSG, Soil Power Sensor:LM27761DSG
- added U4: TPS60400DBV, Soil Power Sensor:TPS60400DBV
- C10, C6: value 4.7uF -> 1uF; MPN CC0603KRX5R7BB475 -> (none)
- C8: MPN CC0603KRX5R7BB105 -> (none)
Connections:
- removed net N$32: C8.1, U8.C1-
- removed net N$44: R10.1, R11.2, U8.VFB
- removed net N$5: C8.2, U8.C1+
- removed net N$53: C10.1, U8.CPOUT
- new net N$10: C6.2, U4.CFLY-
- new net N$7: C6.1, U4.CFLY+
- net +3V3: now also C10.1, U4.IN
- net -3V3: now also C8.1, U4.OUT; no longer C11.1, R10.2, U8.VOUT
- net GND: now also C8.2, U4.GND; no longer C11.2, C6.2, R11.1, U8.GND
- net PC1: no longer U8.EN
- net VCC: no longer C6.1, U8.VIN
Other:
- note added: "Place bypass caps close to package"
- note removed: "Vout = -1.22 (R1 + R2) / R2"
- moved on the sheet: -3V3, C10, C6, C8

Commit message: Closes #9
Parts:
- added U5: FM24CL16B-G, Soil Power Sensor:FM24CL16B-G
Connections:
- net +3V3: now also U5.VDD
- net GND: now also U5.VSS
- net SCL: now also U5.SCL
- net SDA: now also U5.SDA
Other:
- note added: "FRAM"
- note added: "WP (Write Protect) is pulled down internally"
- moved on the sheet: 3V3, D1, R13, R14, U7, X4-1, X4-2, X4-3

Commit message: Closes #12
Parts:
- removed I: TPB1,27, testpad:TPB1,27
Connections:
- removed net PC0: U3A.!PD, U3B.!PD
- new net POWERDOWN: U2.VS, U3A.!PD, U3B.!PD, U7.D9/PA9
- net +3V3: no longer U2.VS
- net N$37: no longer I.TP
Other:
- moved on the sheet: C1, C12, C2, C7, C9, R2, R3, R8, R9, U1, U3A, U3C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
